Commit message: docs: document CAD-based ROS 2 PX4 simulation

File: drone_sim_ws/src/drone_arm_sim/urdf/my_drone_v3/my_drone_cad_formal_dynamic.urdf (robot description, URDF)
Before this commit: robot my_drone_v2_cad_dynamic, 24 links, 23 joints
Links:
- link arm_base_link: mass 0.400642378 -> 0.740718627769
- link base_link: mass 1.35708646 -> 2.509018705
- link gripper_link: mass 0.122292858 -> 0.226098393325
- link lower_arm_link: mass 0.194998025 -> 0.360517702138
- link motor_1_link: mass 0.0287946435 -> 0.0532363274372
- link motor_2_link: mass 0.0287946507 -> 0.0532363407488
- link motor_3_link: mass 0.0287946506 -> 0.0532363405639
- link motor_4_link: mass 0.0287946491 -> 0.0532363377906
- link motor_5_link: mass 0.0287946522 -> 0.053236343522
- link motor_6_link: mass 0.0287946414 -> 0.0532363235547
- link motor_7_link: mass 0.028794653 -> 0.0532363450011
- link motor_8_link: mass 0.0287946478 -> 0.0532363353872
- link moving_jaw_link: mass 0.0707678904 -> 0.130837618649
- link rotor_1_link: mass 0.166991483 -> 0.308738438391
- link rotor_2_link: mass 0.166991541 -> 0.308738545623
- link rotor_3_link: mass 0.166991489 -> 0.308738449484
- link rotor_4_link: mass 0.166991482 -> 0.308738436542
- link rotor_5_link: mass 0.166991518 -> 0.3087385031
- link rotor_6_link: mass 0.166991525 -> 0.308738516042
- link rotor_7_link: mass 0.166991517 -> 0.308738501251
- link rotor_8_link: mass 0.166991498 -> 0.308738466123
- link shoulder_link: mass 0.163253341 -> 0.301827258834
- link upper_arm_link: mass 0.209793591 -> 0.38787215076
- link wrist_link: mass 0.0986089819 -> 0.182310992969

Commit message: feat: add coupled arm flight and PX4 RL validation

File: drone_sim_ws/src/drone_arm_sim/urdf/my_drone_v3/my_drone_cad_formal_dynamic.urdf (robot description, URDF)
Before this commit: robot my_drone_v3_cad_formal_dynamic, 24 links, 23 joints
Links:
- link gripper_link: geometry collision mesh filename=package://drone_arm_sim/meshes/my_drone_v2/visual/so101_gri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 scale=0.001 0.001 0.001; visual mesh filename=package://drone_arm_sim/meshes/my_drone_v2/visual/so101_gri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 scale=0.001 0.001 0.001
- link moving_jaw_link: geometry collision mesh filename=package://drone_arm_sim/meshes/my_drone_v2/visual/so101_mov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 scale=0.001 0.001 0.001; visual mesh filename=package://drone_arm_sim/meshes/my_drone_v2/visual/so101_mov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 scale=0.001 0.001 0.001
