Commit message: fix: add visible landing gear for arm clearance

File: drone_sim_ws/src/drone_arm_sim/urdf/my_drone_v3/my_drone_cad_debug_4kg.urdf (robot description, URDF)
Before this commit: robot my_drone_v3_cad_debug_4kg, 24 links, 23 joints
Links:
- link base_link: geometry collision box size=0.035 0.035 0.817; collision box size=0.035 0.035 0.817

File: drone_sim_ws/src/drone_arm_sim/urdf/my_drone_v3/my_drone_cad_formal_dynamic.urdf (robot description, URDF)
Before this commit: robot my_drone_v3_cad_formal_dynamic, 24 links, 23 joints
Links:
- link base_link: geometry collision box size=0.035 0.035 0.817; collision box size=0.035 0.035 0.817

Commit message: fix: support ground takeoff on retracted arm

File: drone_sim_ws/src/drone_arm_sim/urdf/my_drone_v3/my_drone_cad_debug_4kg.urdf (robot description, URDF)
Before this commit: robot my_drone_v3_cad_debug_4kg, 24 links, 23 joints
Links:
- link arm_base_link: geometry collision box size=0.277366 0.263800 0.111588; visual mesh filename=package://drone_arm_sim/meshes/my_drone_v2/visual/so101_arm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 scale=0.001 0.001 0.001
- link base_link: geometry collision box size=0.32 0.28 0.02; collision box size=0.409830891 0.409830906 0.291000023
- link gripper_link: geometry collision box size=0.060996 0.057342 0.080002; collision mesh filename=package://drone_arm_sim/meshes/my_drone_v2/visual/so101_gri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 scale=0.001 0.001 0.001
- link lower_arm_link: geometry collision box size=0.156642 0.065141 0.037465; visual mesh filename=package://drone_arm_sim/meshes/my_drone_v2/visual/so101_low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 scale=0.001 0.001 0.001
- link moving_jaw_link: geometry collision box size=0.093766 0.115803 0.069980; collision mesh filename=package://drone_arm_sim/meshes/my_drone_v2/visual/so101_mov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 scale=0.001 0.001 0.001
- link shoulder_link: geometry collision box size=0.063497 0.055080 0.110672; visual mesh filename=package://drone_arm_sim/meshes/my_drone_v2/visual/so101_sho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 scale=0.001 0.001 0.001
- link upper_arm_link: geometry collision box size=0.142954 0.067977 0.053988; visual mesh filename=package://drone_arm_sim/meshes/my_drone_v2/visual/so101_upp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 scale=0.001 0.001 0.001
- link wrist_link: geometry collision box size=0.096256 0.076810 0.035863; visual mesh filename=package://drone_arm_sim/meshes/my_drone_v2/visual/so101_wri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 scale=0.001 0.001 0.001

File: drone_sim_ws/src/drone_arm_sim/urdf/my_drone_v3/my_drone_cad_formal_dynamic.urdf (robot description, URDF)
Before this commit: robot my_drone_v3_cad_formal_dynamic, 24 links, 23 joints
Links:
- link arm_base_link: geometry collision box size=0.277366 0.263800 0.111588; visual mesh filename=package://drone_arm_sim/meshes/my_drone_v2/visual/so101_arm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 scale=0.001 0.001 0.001
- link base_link: geometry collision box size=0.32 0.28 0.02; collision box size=0.409830891 0.409830906 0.291000023
- link gripper_link: geometry collision box size=0.060996 0.057342 0.080002; collision mesh filename=package://drone_arm_sim/meshes/my_drone_v2/visual/so101_gri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 scale=0.001 0.001 0.001
- link lower_arm_link: geometry collision box size=0.156642 0.065141 0.037465; visual mesh filename=package://drone_arm_sim/meshes/my_drone_v2/visual/so101_low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 scale=0.001 0.001 0.001
- link moving_jaw_link: geometry collision box size=0.093766 0.115803 0.069980; collision mesh filename=package://drone_arm_sim/meshes/my_drone_v2/visual/so101_mov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 scale=0.001 0.001 0.001
- link shoulder_link: geometry collision box size=0.063497 0.055080 0.110672; visual mesh filename=package://drone_arm_sim/meshes/my_drone_v2/visual/so101_sho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 scale=0.001 0.001 0.001
- link upper_arm_link: geometry collision box size=0.142954 0.067977 0.053988; visual mesh filename=package://drone_arm_sim/meshes/my_drone_v2/visual/so101_upp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 scale=0.001 0.001 0.001
- link wrist_link: geometry collision box size=0.096256 0.076810 0.035863; visual mesh filename=package://drone_arm_sim/meshes/my_drone_v2/visual/so101_wri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 scale=0.001 0.001 0.001

Commit message: make WASD targets deterministic and soften gripper contact

File: drone_sim_ws/src/drone_arm_sim/urdf/my_drone_v3/my_drone_cad_debug_4kg.urdf (robot description, URDF)
Before this commit: robot my_drone_v3_cad_debug_4kg, 24 links, 23 joints
Links:
- link moving_jaw_link: geometry collision box size=0.015 0.015 0.015; collision mesh filename=package://drone_arm_sim/meshes/my_drone_v2/visual/so101_mov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 scale=0.001 0.001 0.001

File: drone_sim_ws/src/drone_arm_sim/urdf/my_drone_v3/my_drone_cad_formal_dynamic.urdf (robot description, URDF)
Before this commit: robot my_drone_v3_cad_formal_dynamic, 24 links, 23 joints
Links:
- link moving_jaw_link: geometry collision box size=0.015 0.015 0.015; collision mesh filename=package://drone_arm_sim/meshes/my_drone_v2/visual/so101_mov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 scale=0.001 0.001 0.001

Commit message: snapshot: preserve 1.3kg directional flight progress

File: drone_sim_ws/src/drone_arm_sim/urdf/my_drone_v3/my_drone_cad_debug_4kg.urdf (robot description, URDF)
Before this commit: robot my_drone_v3_cad_debug_4kg, 24 links, 23 joints
Joints:
- joint elbow_flex: origin xyz=-0.112441148 -0.0015112976 -0.0287159872 rpy=0 0 0 -> xyz=-0.112441148 -0.0015112976 -0.0287159872 rpy=0.0970462031121 1.40596913594 0.0971862997081
- joint shoulder_lift: origin xyz=0.0313169276 0.0135548602 -0.0573278478 rpy=0 0 0 -> xyz=0.0313169276 0.0135548602 -0.0573278478 rpy=-0.0686118073601 -1.4451543931 0.0603617392507
- joint wrist_flex: origin xyz=0.13415811 -0.00208216344 -0.0038220943 rpy=0 0 0 -> xyz=0.13415811 -0.00208216344 -0.0038220943 rpy=-5.34681816356e-07 0.0127093291979 0.000221829007818
- joint wrist_roll: origin xyz=0.0581983646 -0.0171226371 0.000213439633 rpy=0 0 0 -> xyz=0.0581983646 -0.0171226371 0.000213439633 rpy=-0.785362744186 -0.00257767896788 -0.00622469170698
